File: feather_ice40.kicad_pcb (KiCad board)
At the start: 2 copper layers, 50.8 x 22.9 mm, 31 parts, among them J1 USB_OTG, J10 FeatherTop, J2 CONN_01X02, J3 CONN_01X01, J4 CONN_01X01, J5 CONN_01X01, J6 CONN_01X01, J7 CONN_02X05, J9 FeatherBottom, U1 HX4K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

Commit message: Fully routed. Needs silk cleanup.
Parts:
- removed C13: .1uF, Capacitors_SMD:C_0603
- added C1: 0.1uF, Capacitors_SMD:C_0603, F.Cu at (131.1, 67.4)
- added C2: 0.1uF, Capacitors_SMD:C_0603, F.Cu at (120.3, 74.2)
- added C4: 0.1uF, Capacitors_SMD:C_0603, F.Cu at (128.4, 77.0)
- added C5: 0.1uF, Capacitors_SMD:C_0603, F.Cu at (124.9, 79.3)
- added C6: 10uF, Capacitors_SMD:C_0603, F.Cu at (127.4, 78.6)
- added C7: 1uF, Capacitors_SMD:C_0603, F.Cu at (127.9, 66.9)
- added C8: 0.1uF, Capacitors_SMD:C_0603, F.Cu at (127.9, 65.4)
- added D4: Neopixel_THT, LEDs:LED_WS2812B-PLCC4, F.Cu at (133.9, 76.6)
- added J8: Conn_01x04, Pin_Headers:Pin_Header_Straight_1x04_Pitch2.54mm, F.Cu at (140.9, 68.6)
- added R1: 10k, Resistors_SMD:R_0603, F.Cu at (114.3, 67.2)
- added R2: 100, Resistors_SMD:R_0603, F.Cu at (125.5, 77.0)
- added R3: 10k, Resistors_SMD:R_0603, F.Cu at (114.3, 68.9)
- added SW1: SW_SPST, Buttons_Switches_SMD:SW_SPST_KMR2, F.Cu at (99.6, 78.9)
- U1: value HX4K -> ICE40UP5K-SG48; footprint lattice:CB132 -> Housings_DFN_QFN:QFN-48-1EP_7x7mm_Pitch0.5mm
- U2: footprint flash:SOIC-8 -> Housings_SOIC:SOIC-8_3.9x4.9mm_Pitch1.27mm
- U4: value SPX3819M5-L-1-8/TR -> SPX3819M5-L-1-2/TR
- moved U2 17.6 mm to (135.0, 69.8), turned to 90 degrees
- moved U4 11.2 mm to (119.3, 67.0), turned to 0 degrees
- moved C16 10.8 mm to (122.0, 66.3), turned to 270 degrees
- moved R7 4.73 mm to (120.8, 76.4), turned to 270 degrees
- moved R6 4.50 mm to (118.6, 75.8), turned to 180 degrees
- moved U1 3.93 mm to (125.9, 71.9), turned to 270 degrees
- moved C14 2.66 mm to (112.3, 69.6)
- moved U3 2.35 mm to (109.7, 69.1)
- moved C19 2.17 mm to (112.3, 66.4), turned to 270 degrees
- moved R4 1.48 mm to (109.9, 65.8)
Connections:
- C16 pad 1: +1V8 -> +1V2
- J10 pad 11: /riscSCL -> /iceSCL
- J10 pad 12: /riscSDA -> /iceSDA
- J9 pad 1: /riscReset -> /iceReset
- J9 pad 11: /riscSCK -> /iceSCK
- J9 pad 12: /riscMOSI -> /iceMOSI
- J9 pad 13: /riscMISO -> /iceMISO
- J9 pad 14: /riscRX -> /iceRX
- J9 pad 15: /riscTX -> /iceTX
- U2 pad 1: /FLASH_CS -> /flashSS
- U2 pad 2: /FLASH_IO1 -> /flashMISO
- U2 pad 3: /FLASH_IO2 -> +3V3
- U2 pad 5: /FLASH_IO0 -> /flashMOSI
- U2 pad 6: /FLASH_SCK -> /flashSCK
- U2 pad 7: /FLASH_IO3 -> +3V3
- U4 pad 5: +1V8 -> +1V2
- U5 pad 13: /riscReset -> /GCLK4
- U5 pad 14: Net-(U5-Pad14) -> /GCLK5
- U5 pad 15: /riscJTAG_TDO -> /M0TX
- U5 pad 16: /riscJTAG_TCK -> /M0RX
- U5 pad 17: /riscJTAG_TDI -> /configMOSI
- U5 pad 18: /riscJTAG_TMS -> /configSCK
- U5 pad 19: Net-(U5-Pad19) -> /configSS
- U5 pad 20: /riscTX -> /configMISO
- U5 pad 21: /riscRX -> /cdone
- U5 pad 22: Net-(U5-Pad22) -> /iceReset
Routing:
- net +3V3: track 79.0 -> 145.5 mm, vias 2 -> 7
- net +1V2: track 0.00 -> 61.6 mm, vias 0 -> 2
- net /iceReset: track 0.00 -> 53.4 mm, vias 0 -> 4
- net /configSS: track 0.00 -> 52.7 mm, vias 0 -> 2
- net /configSCK: track 0.00 -> 52.4 mm, vias 0 -> 1
- net /configMISO: track 0.00 -> 51.9 mm, vias 0 -> 1
- net /configMOSI: track 0.00 -> 51.3 mm, vias 0 -> 1
- net /riscReset: track 43.4 -> 0.00 mm, vias 4 -> 0
- net /cdone: track 0.00 -> 21.9 mm, vias 0 -> 2
- net /GCLK4: track 0.00 -> 21.8 mm, vias 0 -> 2
- net GND: track 38.1 -> 59.7 mm, vias 8 -> 19
- net /FLASH_IO0: track 18.0 -> 0.00 mm
- net /FLASH_IO3: track 17.6 -> 0.00 mm
- net +1V8: track 15.4 -> 0.00 mm
- net /FLASH_IO1: track 15.2 -> 0.00 mm
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- added copper zone on B.Cu, net GND
- added copper zone on F.Cu, net GND
Other:
- rule pad_to_mask_clearance: 0.2 -> 0.1
- board text added: "CFG"
- board text added: "CK"
- board text added: "CS"
- board text added: "ICE40"
- board text added: "SI"
- board text added: "SO"

Commit message: Silkscreen polish.
Parts:
- moved D3 0.66 mm to (94.6, 67.1), turned to 180 degrees
Routing:
- net GND: track 59.7 -> 63.2 mm
- net Net-(D3-Pad1): track 4.69 -> 1.97 mm
- net /D13: track 34.2 -> 35.1 mm
